File: schematics/relay_board_schematics/Relay_assembly.sch (KiCad schematic (older format))
At the start: 14 parts, among them Q1 MMBF170, Q2 MMBF170, U1 SPST_POWER_RELAY, U2 dpdt_relay, U3 INA180A1, U4 INA180A1

Commit message: Change fusing from bottom side to top side
Correct that error. Also add flyback diode to relay board
Parts:
- added D1, D2: D, Diodes_THT:D_DO-35_SOD27_P7.62mm_Horizontal, symbol D
Connections:
- net +12V: now also D1.1 (K), D2.1 (K)
- net at Q1.3 (D), U1.2 (COUT): now also D1.2 (A)
- net at Q2.3 (D), U2.3 (CIN): now also D2.2 (A)
Changed lines of the file:
@@
 $EndComp
 Wire Wire Line
-	3350 3050 3500 3050
+	3150 3050 3500 3050
 $Comp
 L +12V #PWR018
@@
 	1    0    0    -1
 $EndComp
+$Comp
+L D D1
+U 1 1 5A5EA1E1
+P 3150 2900
+F 0 "D1" H 3150 3000 50  0000 C CNN
+F 1 "D" H 3150 2800 50  0000 C CNN
+F 2 "Diodes_THT:D_DO-35_SOD27_P7.62mm_Horizontal" H 3150 2900 50  0001 C CNN
+F 3 "" H 3150 2900 50  0001 C CNN
+	1    3150 2900
+	0    1    1    0
+$EndComp
+$Comp
+L D D2
+U 1 1 5A5EA2DD
+P 4900 4625
+F 0 "D2" H 4900 4725 50  0000 C CNN
+F 1 "D" H 4900 4525 50  0000 C CNN
+F 2 "Diodes_THT:D_DO-35_SOD27_P7.62mm_Horizontal" H 4900 4625 50  0001 C CNN
+F 3 "" H 4900 4625 50  0001 C CNN
+	1    4900 4625
+	-1   0    0    1
+$EndComp
+Wire Wire Line
+	4750 4500 4750 4625
+Wire Wire Line
+	5050 4625 5050 4500
+Connection ~ 3350 3050
+Wire Wire Line
+	3150 2750 3350 2750
+Connection ~ 3350 2750
 $EndSCHEMATC
