File: schematics/relay_board_schematics/rlcsv2_modular.sch (KiCad schematic (older format))
At the start: 12 parts, among them P1 ACT_PWR, P2 CONN_01X09, P3 ACTUATOR

Commit message: Change fusing from bottom side to top side
Correct that error. Also add flyback diode to relay board
Connections:
- net GND: now also P1.1 (P1); no longer F1.2
- net Relays/VIN: now also F1.2; no longer P1.2 (P2)
- net at F1.1: now also P1.2 (P2); no longer P1.1 (P1)
Other:
- moved on the sheet: F1
Changed lines of the file:
@@
 L FUSE F1
 U 1 1 597C3625
-P 3450 3250
-F 0 "F1" H 3550 3300 50  0000 C CNN
-F 1 "FUSE" H 3350 3200 50  0000 C CNN
-F 2 "custom:littlefuse_01000020Z" H 3450 3250 50  0001 C CNN
-F 3 "" H 3450 3250 50  0000 C CNN
-	1    3450 3250
+P 3575 2900
+F 0 "F1" H 3675 2950 50  0000 C CNN
+F 1 "FUSE" H 3475 2850 50  0000 C CNN
+F 2 "custom:littlefuse_01000020Z" H 3575 2900 50  0001 C CNN
+F 3 "" H 3575 2900 50  0000 C CNN
+	1    3575 2900
 	1    0    0    -1
 $EndComp
@@
 	3200 2500 5050 2500
 Wire Wire Line
-	3200 2900 5050 2900
-Wire Wire Line
 	3200 3000 3200 3250
 Wire Wire Line
-	3700 3250 3850 3250
+	3200 3250 3850 3250
 Wire Wire Line
 	3850 3250 3850 3300
@@
 Wire Wire Line
 	5400 4850 6150 4850
+Wire Wire Line
+	3200 2900 3325 2900
+Wire Wire Line
+	3825 2900 5050 2900
 $EndSCHEMATC
