File: schematics/relay_board_v2_schematics/Relay_assembly.sch (KiCad schematic (older format))
At the start: 16 parts, among them Q1 MMBF170, Q2 MMBF170, U1 SPST_POWER_RELAY, U2 dpdt_relay, U3 INA180A1, U4 INA180A1

Commit message: Add changes for wire cleanup for RLCS
Implement I2C protocol for board communication
Add Dip[ switch, programming header and pic to enable I2C

Signed-off-by: Aidan Ha <qbha@edu.uwaterloo.ca>
Changed lines of the file:
@@
 $Descr A4 11693 8268
 encoding utf-8
-Sheet 2 2
+Sheet 2 3
 Title "RLCSv3"
 Date "2019-10-27"
@@
 $EndComp
 Wire Wire Line
-	5350 3650 6950 3650
-Wire Wire Line
-	5350 3750 7700 3750
+	5350 3650 6850 3650
+Wire Wire Line
+	5350 3750 7600 3750
 Text HLabel 8950 3650 2    60   Input ~ 0
 P1
@@
 G2
 Wire Wire Line
-	7250 3650 8950 3650
-Wire Wire Line
-	8000 3750 8950 3750
+	7250 3650 7400 3650
+Wire Wire Line
+	8000 3750 8050 3750
 Wire Wire Line
 	8050 3100 8050 3750
@@
 $EndComp
 Wire Wire Line
-	3150 3050 3500 3050
+	3150 3050 3350 3050
 $Comp
 L rlcsv3_modular-rescue:+12V #PWR018
@@
 	3350 4500 4750 4500
 Wire Wire Line
-	7600 1300 7600 1750
+	7600 1300 7600 1550
 $Comp
 L rlcsv3_modular-rescue:GND #PWR019
@@
 $EndComp
 Wire Wire Line
-	8250 2250 8250 2700
+	8250 2250 8250 2500
 $Comp
 L rlcsv3_modular-rescue:GND #PWR021
@@
 	2250 5100 2300 5100
 Wire Wire Line
-	2600 5100 3050 5100
+	2600 5100 2650 5100
 $Comp
 L rlcsv3_modular-rescue:R R1
@@
 	2250 3300 2300 3300
 Wire Wire Line
-	2600 3300 3050 3300
+	2600 3300 2650 3300
 Text HLabel 4700 2850 2    60   Input ~ 0
 VIN
@@
 	2250 2500 3350 2500
 Wire Wire Line
-	3350 2500 3350 2850
+	3350 2500 3350 2750
 $Comp
 L rlcsv3_modular-rescue:+12V #PWR022
@@
 	3150 2750 3350 2750
 Connection ~ 3350 2750
+Wire Wire Line
+	2650 5100 3050 5100
+Wire Wire Line
+	2650 3300 3050 3300
+Wire Wire Line
+	8050 3750 8950 3750
+Wire Wire Line
+	7400 3650 8950 3650
+Wire Wire Line
+	6850 3650 6950 3650
+Wire Wire Line
+	7600 3750 7700 3750
+Wire Wire Line
+	7600 1550 7600 1750
+Wire Wire Line
+	8250 2500 8250 2700
+Wire Wire Line
+	3350 3050 3500 3050
+Wire Wire Line
+	3350 2750 3350 2850
 $EndSCHEMATC
