File: schematics/power_board_schematics/test.kicad_pcb (KiCad board)
At the start: 2 copper layers, 124.5 x 101.6 mm, 55 parts, among them J1 SD_Card, J10 Conn_14_to_21, J11 conn_power, J12 conn_A8_to_A15, J13 conn_A0_to_A7, J14 conn_22_to_53, J2 Conn_01x05_Male, J3 Conn_01x05_Male, J4 Battery Conn, J5 CONN_01X02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

Commit message: Made the pcb
Parts:
- J2: footprint Connector_JST:JST_EH_B5B-EH-A_1x05_P2.50mm_Vertical -> Connectors_Terminal_Blocks:TerminalBlock_Pheonix_MKDS1.5-2pol
- J3: footprint Connector_JST:JST_EH_B5B-EH-A_1x05_P2.50mm_Vertical -> Connectors_Molex:Molex_KK-6410-02_02x2.54mm_Straight
- J9: footprint Connector_PinHeader_2.54mm:PinHeader_1x10_P2.54mm_Vertical -> Connector_PinSocket_2.54mm:PinSocket_1x08_P2.54mm_Vertical
- moved S1 89.2 mm to (135.9, 71.1), turned to 0 degrees
- moved J9 57.1 mm to (96.5, 100.3)
- moved J13 54.0 mm to (143.5, 120.7)
- moved J8 54.0 mm to (96.5, 72.4)
- moved J12 52.9 mm to (144.8, 96.5)
- moved J11 49.5 mm to (146.1, 71.1)
- moved J10 48.4 mm to (96.5, 124.5)
- moved J3 30.0 mm to (102.9, 154.9)
- moved R11 23.7 mm to (114.3, 88.9), turned to 270 degrees
- moved J2 23.2 mm to (104.1, 142.1), turned to 90 degrees
- moved TP2 16.2 mm to (114.3, 109.2)
- moved R7 14.5 mm to (128.3, 83.8), turned to 180 degrees
- moved J4 13.5 mm to (118.1, 148.6)
- moved R3 11.4 mm to (139.7, 90.2), turned to 270 degrees
- moved R6 11.4 mm to (137.2, 90.2)
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Routing:
- net GND: track 0.00 -> 217.9 mm, vias 0 -> 6
- net +5V: track 0.00 -> 176.6 mm
- net +12V: track 0.00 -> 77.3 mm
- net +3V3: track 0.00 -> 55.2 mm, vias 0 -> 1
- net Net-(F1-Pad1): track 0.00 -> 32.1 mm
- net Net-(J1-Pad2): track 0.00 -> 26.6 mm
- net Net-(J1-Pad1): track 0.00 -> 24.1 mm
- net ARD_CON_SD_CD: track 0.00 -> 22.9 mm, vias 0 -> 1
- net Net-(J1-Pad8): track 0.00 -> 22.9 mm, vias 0 -> 1
- net /SCL: track 0.00 -> 18.7 mm
- net Net-(J11-Pad2): track 0.00 -> 16.8 mm
- net Net-(J1-Pad5): track 0.00 -> 15.4 mm, vias 0 -> 1
- net Net-(J11-Pad6): track 0.00 -> 15.1 mm
- net Net-(AFF1-Pad9): track 0.00 -> 14.9 mm
- net Net-(AFF1-Pad4): track 0.00 -> 14.2 mm, vias 0 -> 1
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Other:
- board size 124.5 x 101.6 mm -> 121.9 x 101.6 mm
- board text added: "+"
- board text added: "+12v-"
- board text added: "+5v-"
- board text added: "-"
- board text added: "0v"
- board text added: "BATT + -"
