File: schematics/power_board_schematics/rlcs_power.sch (KiCad schematic (older format))
At the start: 39 parts, among them J1 SD_Card, J2 Battery Conn, J3 CONN_01X02, J4 CONN_01X02, J6 CONN_01X02, Q4 Q_NPN_BEC, Q5 Q_NPN_BEC, T1 12 to 3v3, T2 12 to 5

Commit message: third commit, mainly made it more consistent
Parts:
- removed ~: conn_5, symbol custom:conn_5
- added U1, U2: Conn_01x05_Male, symbol Connector:Conn_01x05_Male
Connections:
- net +12P is gone; now on net +12V: C1.1, C2.1, F1.2, J6.1 (P1), T1.1 (Vin), T2.1 (Vin), TP3.1
- net +12V: now also U1.4 (Pin_4), U1.5 (Pin_5), U2.4 (Pin_4), U2.5 (Pin_5)
- net GND: now also U1.3 (Pin_3), U2.3 (Pin_3)
- net SCL: now also U1.2 (Pin_2), U2.2 (Pin_2)
- net SDA: now also U1.1 (Pin_1), U2.1 (Pin_1)
- net Sevenseg_G: now reaches R2.1
- net Sevenseg_F: now reaches R3.1
- net Sevenseg_E: now reaches R4.1
- net Sevenseg_D: now reaches R5.1
- net Sevenseg_C: now reaches R6.1
- net Sevenseg_B: now reaches R7.1
- net Sevenseg_A: now reaches R8.1
- net Sevenseg_DP: now reaches R9.1
Changed lines of the file:
@@
-$EndComp
-$Comp
-L power:+12P #PWR03
-U 1 1 59B5C82D
-P 9600 1800
-F 0 "#PWR03" H 9600 1650 50  0001 C CNN
-F 1 "+12P" H 9600 1940 50  0000 C CNN
-F 2 "" H 9600 1800 50  0001 C CNN
-F 3 "" H 9600 1800 50  0001 C CNN
-	1    9600 1800
-	1    0    0    -1
 $EndComp
 $Comp
@@
 F 3 "" H 8300 3450 50  0001 C CNN
 	1    8300 3450
-	1    0    0    -1
-$EndComp
-$Comp
-L power:+12P #PWR05
-U 1 1 59B5CE01
-P 7850 3100
-F 0 "#PWR05" H 7850 2950 50  0001 C CNN
-F 1 "+12P" H 7850 3240 50  0000 C CNN
-F 2 "" H 7850 3100 50  0001 C CNN
-F 3 "" H 7850 3100 50  0001 C CNN
-	1    7850 3100
 	1    0    0    -1
 $EndComp
@@
 	1    0    0    -1
 $EndComp
-$Sheet
-S 900  7100 1150 600
-U 59C6DB4C
-F0 "Arduino Connections" 60
-F1 "ardconn.sch" 60
-$EndSheet
 Text GLabel 1950 1250 0    60   Input ~ 0
 ARD_CON_SD_SS
@@
 $EndComp
 $Comp
-L power:+12P #PWR021
-U 1 1 59C9B4D2
-P 9900 4150
-F 0 "#PWR021" H 9900 4000 50  0001 C CNN
-F 1 "+12P" H 9900 4290 50  0000 C CNN
-F 2 "" H 9900 4150 50  0001 C CNN
-F 3 "" H 9900 4150 50  0001 C CNN
-	1    9900 4150
-	1    0    0    -1
-$EndComp
-$Comp
 L Device:Q_NPN_BEC Q5
 U 1 1 59CA20EF
@@
 	0    -1   -1   0
 $EndComp
-Text Notes 3200 4800 0    60   ~ 0
-100ohm\nresistors\n
 $Comp
 L Device:R_Small R2
@@
 ARD_CON_7SEG_D1
 $Comp
-L custom:conn_5 ~
-U 1 1 5ECEAAD4
-P 6750 4850
-F 0 "~" H 6708 5497 60  0000 C CNN
-F 1 "conn_5" H 6708 5391 60  0000 C CNN
-F 2 "" H 6750 5450 60  0001 C CNN
-F 3 "" H 6750 5450 60  0001 C CNN
-	1    6750 4850
-	1    0    0    -1
-$EndComp
-Wire Wire Line
-	7150 5350 7150 4850
-Wire Wire Line
-	6800 5350 7150 5350
-Wire Wire Line
-	7550 3750 7650 3750
-Wire Wire Line
-	6800 4850 7150 4850
-Connection ~ 7150 4850
-Wire Wire Line
-	7150 4850 7150 3900
-$Comp
 L power:+12V #PWR?
-U 1 1 5ED2A677
-P 7150 3900
-F 0 "#PWR?" H 7150 3750 50  0001 C CNN
-F 1 "+12V" H 7165 4073 50  0000 C CNN
-F 2 "" H 7150 3900 50  0001 C CNN
-F 3 "" H 7150 3900 50  0001 C CNN
-	1    7150 3900
-	1    0    0    -1
-$EndComp
-$Comp
-L power:+5V #PWR?
-U 1 1 5ED2ACA3
-P 7350 3900
-F 0 "#PWR?" H 7350 3750 50  0001 C CNN
-F 1 "+5V" H 7365 4073 50  0000 C CNN
-F 2 "" H 7350 3900 50  0001 C CNN
-F 3 "" H 7350 3900 50  0001 C CNN
-	1    7350 3900
-	1    0    0    -1
-$EndComp
-Wire Wire Line
-	6800 5050 7750 5050
-Wire Wire Line
-	6800 5150 7550 5150
-Wire Wire Line
-	6800 5250 7350 5250
-Wire Wire Line
-	7350 3900 7350 4750
-Wire Wire Line
-	7550 3750 7550 4650
-Wire Wire Line
-	6800 4750 7350 4750
-Connection ~ 7350 4750
-Wire Wire Line
-	7350 4750 7350 5250
-Wire Wire Line
-	6800 4650 7550 4650
-Connection ~ 7550 4650
-Wire Wire Line
-	7550 4650 7550 5150
+U 1 1 5ED7013C
+P 9900 4150
+F 0 "#PWR?" H 9900 4000 50  0001 C CNN
+F 1 "+12V" H 9915 4323 50  0000 C CNN
+F 2 "" H 9900 4150 50  0001 C CNN
+F 3 "" H 9900 4150 50  0001 C CNN
+	1    9900 4150
+	1    0    0    -1
+$EndComp
+$Comp
+L power:+12V #PWR?
+U 1 1 5ED78628
+P 9600 1800
+F 0 "#PWR?" H 9600 1650 50  0001 C CNN
+F 1 "+12V" H 9615 1973 50  0000 C CNN
+F 2 "" H 9600 1800 50  0001 C CNN
+F 3 "" H 9600 1800 50  0001 C CNN
+	1    9600 1800
+	1    0    0    -1
+$EndComp
+$Comp
+L power:+12V #PWR?
+U 1 1 5ED86EA7
+P 7850 3100
+F 0 "#PWR?" H 7850 2950 50  0001 C CNN
+F 1 "+12V" H 7865 3273 50  0000 C CNN
+F 2 "" H 7850 3100 50  0001 C CNN
+F 3 "" H 7850 3100 50  0001 C CNN
+	1    7850 3100
+	1    0    0    -1
+$EndComp
+$Sheet
+S 900  7100 1150 600
+U 59C6DB4C
+F0 "Arduino Connections" 60
+F1 "ardconn.sch" 60
+$EndSheet
+Text GLabel 2500 5850 0    60   Input ~ 0
+Sevenseg_DP
+Text GLabel 2500 4650 0    60   Input ~ 0
+Sevenseg_F
+Text GLabel 2500 5050 0    60   Input ~ 0
+Sevenseg_D
+Text GLabel 2500 5250 0    60   Input ~ 0
+Sevenseg_C
+Text GLabel 2500 5450 0    60   Input ~ 0
+Sevenseg_B
+Text GLabel 2500 5650 0    60   Input ~ 0
+Sevenseg_A
+Text GLabel 2500 4850 0    60   Input ~ 0
+Sevenseg_E
+Text GLabel 2500 4450 0    60   Input ~ 0
+Sevenseg_G
+Text Notes 3200 4800 0    60   ~ 0
+100ohm\nresistors\n
+Wire Wire Line
+	3350 4900 3150 4900
+Wire Wire Line
+	3150 4900 3150 4450
+Wire Wire Line
+	2500 4450 3150 4450
+Wire Wire Line
+	3350 5000 3000 5000
+Wire Wire Line
+	3000 5000 3000 4650
+Wire Wire Line
+	3000 4650 2500 4650
+Wire Wire Line
+	3350 5100 2850 5100
+Wire Wire Line
+	2850 5100 2850 4850
+Wire Wire Line
+	2850 4850 2500 4850
+Wire Wire Line
+	3350 5200 2750 5200
+Wire Wire Line
+	2750 5200 2750 5050
+Wire Wire Line
+	2750 5050 2500 5050
+Wire Wire Line
+	3350 5300 2700 5300
+Wire Wire Line
+	2700 5300 2700 5250
+Wire Wire Line
+	2700 5250 2500 5250
+Wire Wire Line
+	3350 5400 2600 5400
+Wire Wire Line
+	2600 5400 2600 5450
+Wire Wire Line
+	2600 5450 2500 5450
+Wire Wire Line
+	3350 5500 2650 5500
+Wire Wire Line
+	2650 5500 2650 5650
+Wire Wire Line
+	2650 5650 2500 5650
+Wire Wire Line
+	3350 5750 2650 5750
+Wire Wire Line
+	2650 5750 2650 5850
+Wire Wire Line
+	2650 5850 2500 5850
+Wire Wire Line
+	7750 4750 7750 5250
+Text Label 7750 4750 0    60   ~ 0
+SDA
+Text Label 7650 4650 0    60   ~ 0
+SCL
+Wire Wire Line
+	7550 4350 7550 4450
+Wire Wire Line
+	7650 4850 7650 5350
+Wire Wire Line
+	7750 5250 6700 5250
+Connection ~ 7450 4950
+Wire Wire Line
+	7450 4950 7450 5450
+Connection ~ 7250 5050
+Wire Wire Line
+	7250 5050 7250 5550
+Connection ~ 7050 5150
+Wire Wire Line
+	7050 5150 7050 5650
+Wire Wire Line
+	6700 4750 7750 4750
+Wire Wire Line
+	6700 4850 7650 4850
+Wire Wire Line
+	7450 4950 7450 4350
+Wire Wire Line
+	6700 4950 7450 4950
+Wire Wire Line
+	7250 5050 6700 5050
+Wire Wire Line
+	7250 4450 7250 5050
+Wire Wire Line
+	7050 5150 7050 4450
+Wire Wire Line
+	6700 5150 7050 5150
+Wire Wire Line
+	7450 4350 7550 4350
+Wire Wire Line
+	7050 5650 6700 5650
+Wire Wire Line
+	7250 5550 6700 5550
+Wire Wire Line
+	7450 5450 6700 5450
+Wire Wire Line
+	7650 5350 6700 5350
+Connection ~ 7650 4850
+Wire Wire Line
+	7650 4850 7650 4650
+$Comp
+L Connector:Conn_01x05_Male U2
+U 1 1 5EE7917B
+P 6500 5450
+F 0 "U2" H 6100 5650 50  0000 C CNN
+F 1 "Conn_01x05_Male" H 6100 5500 50  0000 C CNN
+F 2 "" H 6500 5450 50  0001 C CNN
+F 3 "~" H 6500 5450 50  0001 C CNN
+	1    6500 5450
+	1    0    0    -1
+$EndComp
+$Comp
+L power:+12V #PWR?
+U 1 1 5EE7C608
+P 7050 4450
+F 0 "#PWR?" H 7050 4300 50  0001 C CNN
+F 1 "+12V" H 7065 4623 50  0000 C CNN
+F 2 "" H 7050 4450 50  0001 C CNN
+F 3 "" H 7050 4450 50  0001 C CNN
+	1    7050 4450
+	1    0    0    -1
+$EndComp
+$Comp
+L power:+12V #PWR?
+U 1 1 5EE7D5D1
+P 7250 4450
+F 0 "#PWR?" H 7250 4300 50  0001 C CNN
+F 1 "+12V" H 7265 4623 50  0000 C CNN
+F 2 "" H 7250 4450 50  0001 C CNN
+F 3 "" H 7250 4450 50  0001 C CNN
+	1    7250 4450
+	1    0    0    -1
+$EndComp
 $Comp
 L power:GND #PWR?
-U 1 1 5ED75BA3
-P 7650 3750
-F 0 "#PWR?" H 7650 3500 50  0001 C CNN
-F 1 "GND" H 7655 3577 50  0000 C CNN
-F 2 "" H 7650 3750 50  0001 C CNN
-F 3 "" H 7650 3750 50  0001 C CNN
-	1    7650 3750
-	1    0    0    -1
-$EndComp
-Wire Wire Line
-	6800 4550 7750 4550
-Wire Wire Line
-	7750 4550 7750 5050
-Wire Wire Line
-	6800 4450 7950 4450
-Wire Wire Line
-	7950 4450 7950 4950
-Wire Wire Line
-	7950 4950 6800 4950
-Text Label 7750 4300 0    60   ~ 0
-SCL
-Text Label 7950 4450 0    60   ~ 0
-SDA
-Wire Wire Line
-	7750 4550 7750 4300
-Connection ~ 7750 4550
+U 1 1 5EE7EB92
+P 7550 4450
+F 0 "#PWR?" H 7550 4200 50  0001 C CNN
+F 1 "GND" H 7555 4277 50  0000 C CNN
+F 2 "" H 7550 4450 50  0001 C CNN
+F 3 "" H 7550 4450 50  0001 C CNN
+	1    7550 4450
+	1    0    0    -1
+$EndComp
+$Comp
+L Connector:Conn_01x05_Male U1
+U 1 1 5EE77E1A
+P 6500 4950
+F 0 "U1" H 6100 5050 50  0000 C CNN
+F 1 "Conn_01x05_Male" H 6100 4950 50  0000 C CNN
+F 2 "" H 6500 4950 50  0001 C CNN
+F 3 "~" H 6500 4950 50  0001 C CNN
+	1    6500 4950
+	1    0    0    -1
+$EndComp
 $EndSCHEMATC

Commit message: Fixed the reference designators
Parts:
- renumbered J1 to J0, J6 to J10, J4 to J11, J3 to J12, U1 to J8, U2 to J9
Connections:
- net +12V: no longer J8.4 (Pin_4), J9.4 (Pin_4)
- net +5V: now also J8.4 (Pin_4), J9.4 (Pin_4)
Changed lines of the file:
@@
 $EndComp
 $Comp
-L rlcs_power-rescue:SD_Card J1
+L rlcs_power-rescue:SD_Card J0
 U 1 1 59B5C3D6
 P 5750 2400
-F 0 "J1" H 5100 2950 50  0000 C CNN
+F 0 "J0" H 5100 2950 50  0000 C CNN
 F 1 "SD_Card" H 6350 1850 50  0000 C CNN
 F 2 "rlcs_power:SDCARD" H 5950 2750 50  0001 C CNN
@@
 $EndComp
 $Comp
-L rlcs_power-rescue:CONN_01X02 J4
+L rlcs_power-rescue:CONN_01X02 J11
 U 1 1 59C68325
 P 10200 4850
-F 0 "J4" H 10200 5000 50  0000 C CNN
+F 0 "J11" H 10200 5000 50  0000 C CNN
 F 1 "CONN_01X02" V 10300 4850 50  0000 C CNN
 F 2 "Connectors_Molex:Molex_KK-6410-02_02x2.54mm_Straight" H 10200 4850 50  0001 C CNN
@@
 ARD_CON_SD_WP
 $Comp
-L rlcs_power-rescue:CONN_01X02 J3
+L rlcs_power-rescue:CONN_01X02 J12
 U 1 1 59C7C45A
 P 10200 5450
-F 0 "J3" H 10200 5600 50  0000 C CNN
+F 0 "J12" H 10200 5600 50  0000 C CNN
 F 1 "CONN_01X02" V 10300 5450 50  0000 C CNN
 F 2 "Connectors_Molex:Molex_KK-6410-02_02x2.54mm_Straight" H 10200 5450 50  0001 C CNN
@@
 $EndComp
 $Comp
-L rlcs_power-rescue:CONN_01X02 J6
+L rlcs_power-rescue:CONN_01X02 J10
 U 1 1 59C9B3FF
 P 10200 4250
-F 0 "J6" H 10200 4400 50  0000 C CNN
+F 0 "J10" H 10200 4400 50  0000 C CNN
 F 1 "CONN_01X02" V 10300 4250 50  0000 C CNN
 F 2 "Connectors_Molex:Molex_KK-6410-02_02x2.54mm_Straight" H 10200 4250 50  0001 C CNN
@@
 	7650 4850 7650 4650
 $Comp
-L Connector:Conn_01x05_Male U2
+L Connector:Conn_01x05_Male J9
 U 1 1 5EE7917B
 P 6500 5450
-F 0 "U2" H 6100 5650 50  0000 C CNN
+F 0 "J9" H 6100 5650 50  0000 C CNN
 F 1 "Conn_01x05_Male" H 6100 5500 50  0000 C CNN
 F 2 "" H 6500 5450 50  0001 C CNN
@@
 $EndComp
 $Comp
-L power:+12V #PWR?
-U 1 1 5EE7D5D1
-P 7250 4450
-F 0 "#PWR?" H 7250 4300 50  0001 C CNN
-F 1 "+12V" H 7265 4623 50  0000 C CNN
-F 2 "" H 7250 4450 50  0001 C CNN
-F 3 "" H 7250 4450 50  0001 C CNN
-	1    7250 4450
-	1    0    0    -1
-$EndComp
-$Comp
 L power:GND #PWR?
 U 1 1 5EE7EB92
@@
 $EndComp
 $Comp
-L Connector:Conn_01x05_Male U1
+L Connector:Conn_01x05_Male J8
 U 1 1 5EE77E1A
 P 6500 4950
-F 0 "U1" H 6100 5050 50  0000 C CNN
+F 0 "J8" H 6100 5050 50  0000 C CNN
 F 1 "Conn_01x05_Male" H 6100 4950 50  0000 C CNN
 F 2 "" H 6500 4950 50  0001 C CNN
@@
 	1    0    0    -1
 $EndComp
+$Comp
+L power:+5V #PWR?
+U 1 1 5EE5F18B
+P 7250 4450
+F 0 "#PWR?" H 7250 4300 50  0001 C CNN
+F 1 "+5V" H 7265 4623 50  0000 C CNN
+F 2 "" H 7250 4450 50  0001 C CNN
+F 3 "" H 7250 4450 50  0001 C CNN
+	1    7250 4450
+	1    0    0    -1
+$EndComp

Commit message: Made the pcb
Parts:
- C1: footprint Capacitors_SMD:C_0805_HandSoldering -> Capacitor_SMD:C_0805_2012Metric_Pad1.15x1.40mm_HandSolder
- C2: renamed from C3; footprint Capacitors_SMD:C_0805_HandSoldering -> Capacitor_SMD:C_0805_2012Metric_Pad1.15x1.40mm_HandSolder
- C3: renamed from C2; footprint Capacitors_SMD:C_0805_HandSoldering -> Capacitor_SMD:C_0805_2012Metric_Pad1.15x1.40mm_HandSolder
- C4: renamed from C5; footprint Capacitors_SMD:C_0805_HandSoldering -> Capacitor_SMD:C_0805_2012Metric_Pad1.15x1.40mm_HandSolder
- J1: renamed from J0; footprint rlcs_power:SDCARD -> rlcs_power_footprints:SDCARD
- J2: renamed from J8; footprint (none) -> Connector_JST:JST_EH_B5B-EH-A_1x05_P2.50mm_Vertical
- J3: renamed from J9; footprint (none) -> Connector_JST:JST_EH_B5B-EH-A_1x05_P2.50mm_Vertical
- J4: renamed from J2; footprint Connectors_Terminal_Blocks:TerminalBlock_Pheonix_MKDS1.5-2pol -> TerminalBlock_Phoenix:TerminalBlock_Phoenix_MKDS-1,5-2_1x02_P5.00mm_Horizontal
- J5: renamed from J10; footprint Connectors_Molex:Molex_KK-6410-02_02x2.54mm_Straight -> Connector_Molex:Molex_KK-254_AE-6410-02A_1x02_P2.54mm_Vertical
- J6: renamed from J11; footprint Connectors_Molex:Molex_KK-6410-02_02x2.54mm_Straight -> Connector_Molex:Molex_KK-254_AE-6410-02A_1x02_P2.54mm_Vertical
- J7: renamed from J12; footprint Connectors_Molex:Molex_KK-6410-02_02x2.54mm_Straight -> Connector_Molex:Molex_KK-254_AE-6410-02A_1x02_P2.54mm_Vertical
- JP1: footprint Pin_Headers:Pin_Header_Straight_1x03_Pitch2.54mm -> Connector_PinHeader_2.54mm:PinHeader_1x03_P2.54mm_Horizontal
- Q1: renamed from Q4; footprint TO_SOT_Packages_SMD:SOT-23_Handsoldering -> Package_TO_SOT_SMD:SOT-23-5_HandSoldering
- Q2: renamed from Q5; footprint TO_SOT_Packages_SMD:SOT-23_Handsoldering -> Package_TO_SOT_SMD:SOT-23-5_HandSoldering
- R1: renamed from R24; footprint Resistors_SMD:R_0805_HandSoldering -> Resistor_SMD:R_0805_2012Metric_Pad1.15x1.40mm_HandSolder
- R10: renamed from R5; footprint Resistors_SMD:R_0805_HandSoldering -> Resistor_SMD:R_0805_2012Metric_Pad1.15x1.40mm_HandSolder
- R11: renamed from R6; footprint Resistors_SMD:R_0805_HandSoldering -> Resistor_SMD:R_0805_2012Metric_Pad1.15x1.40mm_HandSolder
- R12: renamed from R7; footprint Resistors_SMD:R_0805_HandSoldering -> Resistor_SMD:R_0805_2012Metric_Pad1.15x1.40mm_HandSolder
- R13: renamed from R8; footprint Resistors_SMD:R_0805_HandSoldering -> Resistor_SMD:R_0805_2012Metric_Pad1.15x1.40mm_HandSolder
- R14: renamed from R9; footprint Resistors_SMD:R_0805_HandSoldering -> Resistor_SMD:R_0805_2012Metric_Pad1.15x1.40mm_HandSolder
- R15: renamed from R10; footprint Resistors_SMD:R_0805_HandSoldering -> Resistor_SMD:R_0805_2012Metric_Pad1.15x1.40mm_HandSolder
- R16: renamed from R11; footprint Resistors_SMD:R_0805_HandSoldering -> Resistor_SMD:R_0805_2012Metric_Pad1.15x1.40mm_HandSolder
- R17: renamed from R26; footprint Resistors_SMD:R_0805_HandSoldering -> Resistor_SMD:R_0805_2012Metric_Pad1.15x1.40mm_HandSolder
- R18: renamed from R27; footprint Resistors_SMD:R_0805_HandSoldering -> Resistor_SMD:R_0805_2012Metric_Pad1.15x1.40mm_HandSolder
- R2: renamed from R1; footprint Resistors_SMD:R_0805_HandSoldering -> Resistor_SMD:R_0805_2012Metric_Pad1.15x1.40mm_HandSolder
- R3: renamed from R12; footprint Resistors_SMD:R_0805_HandSoldering -> Resistor_SMD:R_0805_2012Metric_Pad1.15x1.40mm_HandSolder
- R4: renamed from R13; footprint Resistors_SMD:R_0805_HandSoldering -> Resistor_SMD:R_0805_2012Metric_Pad1.15x1.40mm_HandSolder
- R5: renamed from R14; footprint Resistors_SMD:R_0805_HandSoldering -> Resistor_SMD:R_0805_2012Metric_Pad1.15x1.40mm_HandSolder
- R6: renamed from R15; footprint Resistors_SMD:R_0805_HandSoldering -> Resistor_SMD:R_0805_2012Metric_Pad1.15x1.40mm_HandSolder
- R7: renamed from R2; footprint Resistors_SMD:R_0805_HandSoldering -> Resistor_SMD:R_0805_2012Metric_Pad1.15x1.40mm_HandSolder
- R8: renamed from R3; footprint Resistors_SMD:R_0805_HandSoldering -> Resistor_SMD:R_0805_2012Metric_Pad1.15x1.40mm_HandSolder
- R9: renamed from R4; footprint Resistors_SMD:R_0805_HandSoldering -> Resistor_SMD:R_0805_2012Metric_Pad1.15x1.40mm_HandSolder
- T1, T2: footprint rlcs_power:VXO78XX-1000 -> rlcs_power_footprints:VXO78XX-1000
- TP1: renamed from TP3; footprint Socket_Strips:Socket_Strip_Straight_1x01_Pitch2.00mm -> Connector_PinSocket_2.00mm:PinSocket_1x01_P2.00mm_Vertical
- TP2: footprint Socket_Strips:Socket_Strip_Straight_1x01_Pitch2.00mm -> Connector_PinSocket_2.00mm:PinSocket_1x01_P2.00mm_Vertical
- TP3: renamed from TP0; footprint Socket_Strips:Socket_Strip_Straight_1x01_Pitch2.00mm -> Connector_PinSocket_2.00mm:PinSocket_1x01_P2.00mm_Vertical
- TP4: renamed from TP1; footprint Socket_Strips:Socket_Strip_Straight_1x01_Pitch2.00mm -> Connector_PinSocket_2.00mm:PinSocket_1x01_P2.00mm_Vertical

Commit message: UPdated pcb
Parts:
- JP1: footprint Connector_PinHeader_2.54mm:PinHeader_1x03_P2.54mm_Horizontal -> Connector_PinSocket_2.54mm:PinSocket_1x03_P2.54mm_Vertical_SMD_Pin1Left
Changed lines of the file:
@@
 F 0 "JP1" H 3550 1150 50  0000 L CNN
 F 1 "Jumper_NC_Dual" H 3500 1350 50  0000 C BNN
-F 2 "Connector_PinHeader_2.54mm:PinHeader_1x03_P2.54mm_Horizontal" H 3500 1250 50  0001 C CNN
+F 2 "Connector_PinSocket_2.54mm:PinSocket_1x03_P2.54mm_Vertical_SMD_Pin1Left" H 3500 1250 50  0001 C CNN
 F 3 "" H 3500 1250 50  0001 C CNN
 	1    3500 1250

Commit message: Updated PCB, still need to edit traces
Parts:
- JP1: footprint Connector_PinSocket_2.54mm:PinSocket_1x03_P2.54mm_Vertical_SMD_Pin1Left -> Connector_PinHeader_2.54mm:PinHeader_1x03_P2.54mm_Vertical
Changed lines of the file:
@@
 F 0 "JP1" H 3550 1150 50  0000 L CNN
 F 1 "Jumper_NC_Dual" H 3500 1350 50  0000 C BNN
-F 2 "Connector_PinSocket_2.54mm:PinSocket_1x03_P2.54mm_Vertical_SMD_Pin1Left" H 3500 1250 50  0001 C CNN
+F 2 "Connector_PinHeader_2.54mm:PinHeader_1x03_P2.54mm_Vertical" H 3500 1250 50  0001 C CNN
 F 3 "" H 3500 1250 50  0001 C CNN
 	1    3500 1250
