File: schematics/power_board_schematics/ardconn.sch (KiCad schematic (older format))
At the start: 8 parts, among them J10 Conn_14_to_21, J11 conn_power, J12 conn_A8_to_A15, J13 conn_A0_to_A7, J14 conn_22_to_53, J8 Conn_0_to_7, J9 conn_8_to_13

Commit message: Fix 7 segement display pins to make routing easier and fix footprints
Connections:
- net Sevenseg_B: now also J14.43 (Pin_22); no longer J14.40 (Pin_40)
- net Sevenseg_C: now also J14.38 (Pin_38); no longer J14.43 (Pin_22)
- net Sevenseg_D: now also J14.46 (Pin_46); no longer J14.45 (Pin_24)
- net Sevenseg_D1: now also J14.44 (Pin_44); no longer J14.47 (Pin_26)
- net Sevenseg_D2: now also J14.41 (Pin_20); no longer J14.46 (Pin_46)
- net Sevenseg_DP: now also J14.40 (Pin_40); no longer J14.44 (Pin_44)
- net Sevenseg_F: now also J14.47 (Pin_26); no longer J14.41 (Pin_20)
- net Sevenseg_G: now also J14.45 (Pin_24); no longer J14.38 (Pin_38)
Changed lines of the file:
@@
 EESchema Schematic File Version 4
-LIBS:rlcs_power-cache
 EELAYER 30 0
 EELAYER END
@@
 Text Notes 700  950  0    60   ~ 0
 Arudino Pins 0 - 7
-Text GLabel 9000 3000 2    60   Input ~ 0
-ARD_CON_SD_MOSI
-Text GLabel 7100 3000 0    60   Input ~ 0
-ARD_CON_SD_MISO
-Text GLabel 9000 3200 2    60   Input ~ 0
-ARD_CON_SD_SS
 Text Notes 850  6200 0    60   ~ 0
 All Arduino connections put on this sheet\nso they can be reordered without screwing\nup the main sheet\n\n(this doesn't include power out)
-Text GLabel 7100 3200 0    60   Input ~ 0
-ARD_CON_SD_CD
-Text GLabel 9000 3350 2    60   Input ~ 0
-ARD_CON_SD_WP
 Text GLabel 2450 3800 2    60   Input ~ 0
 ARD_CON_SD_SCL
@@
 Wire Wire Line
 	4700 3250 4450 3250
-Text GLabel 9000 2200 2    60   Input ~ 0
-Sevenseg_F
-Text GLabel 9000 2600 2    60   Input ~ 0
-Sevenseg_D
-Text GLabel 9000 2400 2    60   Input ~ 0
-Sevenseg_C
-Text GLabel 9000 2000 2    60   Input ~ 0
-Sevenseg_A
-Text GLabel 9000 2800 2    60   Input ~ 0
-Sevenseg_D1
-Text GLabel 7100 2800 0    60   Input ~ 0
-Sevenseg_D2
-Text GLabel 7100 2400 0    60   Input ~ 0
-Sevenseg_E
-Text GLabel 7100 2600 0    60   Input ~ 0
-Sevenseg_DP
 Wire Wire Line
 	5100 3250 5250 3250
@@
 Wire Wire Line
 	8700 3000 9000 3000
-Text GLabel 7100 2000 0    60   Input ~ 0
-Sevenseg_G
-Text GLabel 7100 2200 0    60   Input ~ 0
-Sevenseg_B
 Wire Wire Line
 	8300 2600 8750 2600
@@
 	8300 2400 9000 2400
 Wire Wire Line
-	7350 2000 7100 2000
-Wire Wire Line
-	7800 2400 7100 2400
-Wire Wire Line
-	7350 2200 7350 2000
-Wire Wire Line
 	7800 2200 7350 2200
 Wire Wire Line
 	7300 2300 7300 2200
 Wire Wire Line
-	7300 2200 7100 2200
-Wire Wire Line
 	7800 2300 7300 2300
 Wire Wire Line
 	7300 2500 7300 2600
 Wire Wire Line
-	7300 2600 7100 2600
-Wire Wire Line
 	7800 2500 7300 2500
 Wire Wire Line
@@
 Wire Wire Line
 	7800 2600 7350 2600
-Wire Wire Line
-	7350 2800 7100 2800
 Wire Wire Line
 	7800 2800 7400 2800
@@
 Wire Wire Line
 	5250 3250 5250 3650
+Text GLabel 7100 2600 0    60   Input ~ 0
+Sevenseg_D1
+Text GLabel 9000 2000 2    60   Input ~ 0
+Sevenseg_A
+Text GLabel 7100 2000 0    60   Input ~ 0
+Sevenseg_C
+Text GLabel 7100 2800 0    60   Input ~ 0
+Sevenseg_D
+Text GLabel 9000 2800 2    60   Input ~ 0
+Sevenseg_F
+Text GLabel 9000 3350 2    60   Input ~ 0
+ARD_CON_SD_WP
+Text GLabel 9000 3200 2    60   Input ~ 0
+ARD_CON_SD_SS
+Text GLabel 9000 3000 2    60   Input ~ 0
+ARD_CON_SD_MOSI
+Text GLabel 7100 3200 0    60   Input ~ 0
+ARD_CON_SD_CD
+Text GLabel 7100 3000 0    60   Input ~ 0
+ARD_CON_SD_MISO
+Wire Wire Line
+	7350 2200 7350 2000
+Text GLabel 9000 2200 2    60   Input ~ 0
+Sevenseg_D2
+Text GLabel 7100 2400 0    60   Input ~ 0
+Sevenseg_E
+Text GLabel 7100 2200 0    60   Input ~ 0
+Sevenseg_DP
+Text GLabel 9000 2600 2    60   Input ~ 0
+Sevenseg_G
+Text GLabel 9000 2400 2    60   Input ~ 0
+Sevenseg_B
+Wire Wire Line
+	7350 2800 7100 2800
+Wire Wire Line
+	7300 2600 7100 2600
+Wire Wire Line
+	7300 2200 7100 2200
+Wire Wire Line
+	7800 2400 7100 2400
+Wire Wire Line
+	7350 2000 7100 2000
 $EndSCHEMATC

Commit message: Update component placement
Connections:
- net ARD_CON_SD_CD: now also J14.34 (Pin_34); no longer J14.54 (Pin_54)
- net ARD_CON_SD_WP: now also J14.35 (Pin_14); no longer J14.55 (Pin_55)
- net Sevenseg_D2: now also J14.40 (Pin_40); no longer J14.41 (Pin_20)
- net Sevenseg_DP: now also J14.41 (Pin_20); no longer J14.40 (Pin_40)
- net ARD_CON_SDA: now reaches J10.20 (Pin_20)
Changed lines of the file:
@@
 Text Notes 700  2100 0    60   ~ 0
 Arduino Pins 8 - 13 \n+ some others\n
-Text Notes 2800 3150 0    60   ~ 0
-Arduino Pins Power
 Text Notes 700  950  0    60   ~ 0
 Arudino Pins 0 - 7
 Text Notes 850  6200 0    60   ~ 0
 All Arduino connections put on this sheet\nso they can be reordered without screwing\nup the main sheet\n\n(this doesn't include power out)
-Text GLabel 2450 3800 2    60   Input ~ 0
-ARD_CON_SD_SCL
 $Comp
 L custom:conn_22_to_53 J14
@@
 Wire Wire Line
 	8700 1400 8700 1050
-$Comp
-L Switch:SW_Push S1
-U 1 1 5EB5D71A
-P 4900 3250
-F 0 "S1" H 4900 3535 50  0000 C CNN
-F 1 "SW_Push" H 4900 3444 50  0000 C CNN
-F 2 "Button_Switch_SMD:SW_Push_SPST_NO_Alps_SKRK" H 4900 3450 50  0001 C CNN
-F 3 "~" H 4900 3450 50  0001 C CNN
-	1    4900 3250
-	1    0    0    -1
-$EndComp
-Wire Wire Line
-	5250 3650 4450 3650
-Wire Wire Line
-	4700 3250 4450 3250
-Wire Wire Line
-	5100 3250 5250 3250
 Wire Wire Line
 	8750 2800 9000 2800
@@
 	2150 3800 2450 3800
 Wire Wire Line
-	7100 3200 7450 3200
-Wire Wire Line
-	7450 3200 7450 3000
-Wire Wire Line
-	7450 3000 7800 3000
-Wire Wire Line
-	9000 3350 8600 3350
-Wire Wire Line
-	8600 3350 8600 3000
-Wire Wire Line
-	8600 3000 8300 3000
-$Comp
-L custom:conn_power J11
-U 1 1 5ED49DCC
-P 4350 3000
-F 0 "J11" H 4237 3197 60  0000 C CNN
-F 1 "conn_power" H 4237 3091 60  0000 C CNN
-F 2 "Connector_PinSocket_2.54mm:PinSocket_1x08_P2.54mm_Vertical" H 4350 3200 60  0001 C CNN
-F 3 "" H 4350 3200 60  0001 C CNN
-	1    4350 3000
-	1    0    0    -1
-$EndComp
-Wire Wire Line
-	5250 3250 5250 3650
+	7150 1750 7500 1750
 Text GLabel 7100 2600 0    60   Input ~ 0
 Sevenseg_D1
@@
 Text GLabel 9000 2800 2    60   Input ~ 0
 Sevenseg_F
-Text GLabel 9000 3350 2    60   Input ~ 0
+Text GLabel 8850 1750 2    60   Input ~ 0
 ARD_CON_SD_WP
 Text GLabel 9000 3200 2    60   Input ~ 0
@@
 Text GLabel 9000 3000 2    60   Input ~ 0
 ARD_CON_SD_MOSI
-Text GLabel 7100 3200 0    60   Input ~ 0
+Text GLabel 7150 1750 0    60   Input ~ 0
 ARD_CON_SD_CD
 Text GLabel 7100 3000 0    60   Input ~ 0
@@
 Wire Wire Line
 	7350 2200 7350 2000
-Text GLabel 9000 2200 2    60   Input ~ 0
+Text GLabel 7100 2200 0    60   Input ~ 0
 Sevenseg_D2
 Text GLabel 7100 2400 0    60   Input ~ 0
 Sevenseg_E
-Text GLabel 7100 2200 0    60   Input ~ 0
+Text GLabel 9000 2200 2    60   Input ~ 0
 Sevenseg_DP
 Text GLabel 9000 2600 2    60   Input ~ 0
@@
 Wire Wire Line
 	7350 2000 7100 2000
+Wire Wire Line
+	2500 3650 2300 3650
+Wire Wire Line
+	2300 3650 2300 3700
+Wire Wire Line
+	2150 3700 2300 3700
+Text GLabel 2500 3650 2    60   Input ~ 0
+ARD_CON_SDA
+Wire Wire Line
+	5250 3250 5250 3650
+$Comp
+L custom:conn_power J11
+U 1 1 5ED49DCC
+P 4350 3000
+F 0 "J11" H 4237 3197 60  0000 C CNN
+F 1 "conn_power" H 4237 3091 60  0000 C CNN
+F 2 "Connector_PinSocket_2.54mm:PinSocket_1x08_P2.54mm_Vertical" H 4350 3200 60  0001 C CNN
+F 3 "" H 4350 3200 60  0001 C CNN
+	1    4350 3000
+	1    0    0    -1
+$EndComp
+Wire Wire Line
+	5100 3250 5250 3250
+Wire Wire Line
+	4700 3250 4450 3250
+Wire Wire Line
+	5250 3650 4450 3650
+$Comp
+L Switch:SW_Push S1
+U 1 1 5EB5D71A
+P 4900 3250
+F 0 "S1" H 4900 3535 50  0000 C CNN
+F 1 "SW_Push" H 4900 3444 50  0000 C CNN
+F 2 "Button_Switch_SMD:SW_Push_SPST_NO_Alps_SKRK" H 4900 3450 50  0001 C CNN
+F 3 "~" H 4900 3450 50  0001 C CNN
+	1    4900 3250
+	1    0    0    -1
+$EndComp
+Text GLabel 2450 3800 2    60   Input ~ 0
+ARD_CON_SD_SCL
+Text Notes 2800 3150 0    60   ~ 0
+Arduino Pins Power
+Wire Wire Line
+	7500 1750 7500 2000
+Wire Wire Line
+	7500 2000 7800 2000
+Wire Wire Line
+	8850 1750 8550 1750
+Wire Wire Line
+	8550 1750 8550 2000
+Wire Wire Line
+	8550 2000 8300 2000
 $EndSCHEMATC

Commit message: Finish board routing
Connections:
- net ARD_CON_SD_MISO: now also J14.32 (Pin_32); no longer J14.50 (Pin_50)
Changed lines of the file:
@@
 	7800 2600 7350 2600
-Wire Wire Line
-	7800 2800 7400 2800
-Wire Wire Line
-	7400 2800 7400 3000
-Wire Wire Line
-	7400 3000 7100 3000
 Wire Wire Line
 	8300 3100 8350 3100
@@
 Text GLabel 7150 1750 0    60   Input ~ 0
 ARD_CON_SD_CD
-Text GLabel 7100 3000 0    60   Input ~ 0
+Text GLabel 7200 1550 0    60   Input ~ 0
 ARD_CON_SD_MISO
 Wire Wire Line
@@
 Wire Wire Line
 	8550 2000 8300 2000
+Wire Wire Line
+	7200 1550 7600 1550
+Wire Wire Line
+	7600 1550 7600 1900
+Wire Wire Line
+	7600 1900 7800 1900
 $EndSCHEMATC

Commit message: Address Zach comments
Connections:
- net ARD_CON_SD_MISO: now also J14.52 (Pin_52); no longer J14.32 (Pin_32)
- net ARD_CON_SD_MOSI: now also J14.53 (Pin_32); no longer J14.51 (Pin_30)
- net ARD_CON_SD_SS: now also J14.55 (Pin_55); no longer J14.53 (Pin_32)
- net ARD_CON_SD_SCK: now reaches J14.54 (Pin_54)
- net ARD_CON_SD_SCL renamed ARD_CON_SCL
Changed lines of the file:
@@
 	7750 3100 7800 3100
 Wire Wire Line
-	8300 2800 8700 2800
-Wire Wire Line
-	8700 2800 8700 3000
-Wire Wire Line
-	8700 3000 9000 3000
+	8700 3100 9000 3100
 Wire Wire Line
 	8300 2600 8750 2600
@@
 	8300 3100 8350 3100
 Wire Wire Line
-	9000 3200 8650 3200
-Wire Wire Line
-	8650 3200 8650 2900
-Wire Wire Line
-	8650 2900 8300 2900
+	9000 3300 8650 3300
 Wire Wire Line
 	2150 3800 2450 3800
@@
 Text GLabel 8850 1750 2    60   Input ~ 0
 ARD_CON_SD_WP
-Text GLabel 9000 3200 2    60   Input ~ 0
+Text GLabel 9000 3300 2    60   Input ~ 0
 ARD_CON_SD_SS
-Text GLabel 9000 3000 2    60   Input ~ 0
+Text GLabel 9000 3100 2    60   Input ~ 0
 ARD_CON_SD_MOSI
 Text GLabel 7150 1750 0    60   Input ~ 0
 ARD_CON_SD_CD
-Text GLabel 7200 1550 0    60   Input ~ 0
-ARD_CON_SD_MISO
 Wire Wire Line
 	7350 2200 7350 2000
@@
 $EndComp
 Text GLabel 2450 3800 2    60   Input ~ 0
-ARD_CON_SD_SCL
+ARD_CON_SCL
 Text Notes 2800 3150 0    60   ~ 0
 Arduino Pins Power
@@
 	8550 2000 8300 2000
 Wire Wire Line
-	7200 1550 7600 1550
+	8700 2900 8700 3100
 Wire Wire Line
-	7600 1550 7600 1900
+	8650 3300 8650 3000
 Wire Wire Line
-	7600 1900 7800 1900
+	8650 3000 8300 3000
+Wire Wire Line
+	8300 2900 8700 2900
+Wire Wire Line
+	7450 2900 7450 3000
+Wire Wire Line
+	7450 3000 7250 3000
+Wire Wire Line
+	7800 2900 7450 2900
+Text GLabel 7250 3000 0    60   Input ~ 0
+ARD_CON_SD_MISO
+Text GLabel 7200 3200 0    60   Input ~ 0
+ARD_CON_SD_SCK
+Wire Wire Line
+	7800 3000 7500 3000
+Wire Wire Line
+	7500 3000 7500 3200
+Wire Wire Line
+	7500 3200 7200 3200
 $EndSCHEMATC

Commit message: fix silk screens that broke from chaning footprints
Parts:
- S1: footprint Button_Switch_SMD:SW_Push_SPST_NO_Alps_SKRK -> Button_Switch_THT:SW_PUSH_6mm
Changed lines of the file:
@@
 F 0 "S1" H 4900 3535 50  0000 C CNN
 F 1 "SW_Push" H 4900 3444 50  0000 C CNN
-F 2 "Button_Switch_SMD:SW_Push_SPST_NO_Alps_SKRK" H 4900 3450 50  0001 C CNN
+F 2 "Button_Switch_THT:SW_PUSH_6mm" H 4900 3450 50  0001 C CNN
 F 3 "~" H 4900 3450 50  0001 C CNN
 	1    4900 3250
